File: hardware/algyan_8th.es.brd (EAGLE design)
At the start: 130 x 80 mm, 40 parts, among them CN1 4P-2.0, U1 XIAO ESP32C3, U2 TM1640, U3 OSL641501-AY, U4 LTP-12188M-08, U5 NJM2113D, U6 UGSM23A, U7 EC12PLRVF, U8 TVGP01-G73BB, U9 TVGP01-G73BB

Commit message: ES基板の回路図に部品の値を記入
Parts:
- C1: value (none) -> 10u
- C3: value (none) -> DNP
- C7, C8: value 0.01u -> DNP
- R1, R2: value (none) -> 100K
- R10, R11: value 10K -> 0
- R5: value (none) -> 0
- R8, R9: value 10K -> DNP
Changed lines of the file:
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@@
 <setting verticaltext="up"/>
 </settings>
-<grid distance="25" unitdist="mil" unit="mil" style="lines" multiple="4" display="yes" altdistance="0.025" altunitdist="inch" altunit="inch"/>
+<grid distance="25" unitdist="mil" unit="mm" style="lines" multiple="4" display="yes" altdistance="0.025" altunitdist="inch" altunit="inch"/>
 <layers>
 <layer number="1" name="Top" color="4" fill="1" visible="yes" active="yes"/>
@@
 </autorouter>
 <elements>
-<element name="C1" library="rcl" package="C0805" value="" x="60.96" y="60.96" smashed="yes">
+<element name="C1" library="rcl" package="C0805" value="10u" x="60.96" y="60.96" smashed="yes">
 <attribute name="NAME" x="62.865" y="60.96" size="1.016" layer="25" font="vector" ratio="10" align="center-left"/>
 <attribute name="VALUE" x="59.69" y="58.42" size="1.27" layer="27"/>
@@
 <attribute name="NAME" x="50.8" y="22.225" size="1.016" layer="25" font="vector" ratio="10" align="bottom-center"/>
 </element>
-<element name="C3" library="rcl" package="C0805" value="" x="65.405" y="16.51" smashed="yes">
+<element name="C3" library="rcl" package="C0805" value="DNP" x="65.405" y="16.51" smashed="yes">
 <attribute name="NAME" x="67.31" y="16.51" size="1.016" layer="25" font="vector" ratio="10" align="center-left"/>
 <attribute name="VALUE" x="64.135" y="13.97" size="1.27" layer="27"/>
@@
 <attribute name="NAME" x="35.56" y="19.685" size="1.016" layer="25" font="vector" ratio="10" align="bottom-center"/>
 </element>
-<element name="C7" library="rcl" package="C0603" value="0.01u" x="84.455" y="33.02" smashed="yes" rot="R180">
+<element name="C7" library="rcl" package="C0603" value="DNP" x="84.455" y="33.02" smashed="yes" rot="R180">
 <attribute name="NAME" x="86.36" y="33.02" size="1.016" layer="25" font="vector" ratio="10" align="center-left"/>
 </element>
-<element name="C8" library="rcl" package="C0603" value="0.01u" x="78.105" y="33.02" smashed="yes">
+<element name="C8" library="rcl" package="C0603" value="DNP" x="78.105" y="33.02" smashed="yes">
 <attribute name="NAME" x="80.01" y="33.02" size="1.016" layer="25" font="vector" ratio="10" align="center-left"/>
 </element>
@@
 <attribute name="VALUE" x="106.5784" y="66.7004" size="1.27" layer="27" ratio="10" rot="R90"/>
 </element>
-<element name="R1" library="rcl" package="R0603" value="" x="60.96" y="66.04" smashed="yes" rot="R180">
+<element name="R1" library="rcl" package="R0603" value="100K" x="60.96" y="66.04" smashed="yes" rot="R180">
 <attribute name="NAME" x="62.865" y="66.04" size="1.016" layer="25" font="vector" ratio="10" align="center-left"/>
 <attribute name="VALUE" x="61.595" y="67.945" size="1.27" layer="27" rot="R180"/>
 </element>
-<element name="R10" library="rcl" package="R0603" value="10K" x="84.455" y="30.48" smashed="yes">
+<element name="R10" library="rcl" package="R0603" value="0" x="84.455" y="30.48" smashed="yes">
 <attribute name="NAME" x="86.36" y="30.48" size="1.016" layer="25" font="vector" ratio="10" align="center-left"/>
 </element>
-<element name="R11" library="rcl" package="R0603" value="10K" x="78.105" y="30.48" smashed="yes" rot="R180">
+<element name="R11" library="rcl" package="R0603" value="0" x="78.105" y="30.48" smashed="yes" rot="R180">
 <attribute name="NAME" x="80.01" y="30.48" size="1.016" layer="25" font="vector" ratio="10" align="center-left"/>
 </element>
@@
 <attribute name="VALUE" x="116.84" y="27.305" size="1.27" layer="27" rot="R180"/>
 </element>
-<element name="R2" library="rcl" package="R0603" value="" x="60.96" y="63.5" smashed="yes" rot="R180">
+<element name="R2" library="rcl" package="R0603" value="100K" x="60.96" y="63.5" smashed="yes" rot="R180">
 <attribute name="NAME" x="62.865" y="63.5" size="1.016" layer="25" font="vector" ratio="10" align="center-left"/>
 <attribute name="VALUE" x="61.595" y="65.405" size="1.27" layer="27" rot="R180"/>
@@
 <attribute name="NAME" x="50.8" y="24.765" size="1.016" layer="25" font="vector" ratio="10" align="bottom-center"/>
 </element>
-<element name="R5" library="rcl" package="R0603" value="" x="65.405" y="19.05" smashed="yes">
+<element name="R5" library="rcl" package="R0603" value="0" x="65.405" y="19.05" smashed="yes">
 <attribute name="NAME" x="67.31" y="19.05" size="1.016" layer="25" font="vector" ratio="10" align="center-left"/>
 <attribute name="VALUE" x="64.77" y="17.145" size="1.27" layer="27"/>
@@
 <attribute name="VALUE" x="90.17" y="15.24" size="1.27" layer="27" rot="R180"/>
 </element>
-<element name="R8" library="rcl" package="R0603" value="10K" x="84.455" y="27.94" smashed="yes">
+<element name="R8" library="rcl" package="R0603" value="DNP" x="84.455" y="27.94" smashed="yes">
 <attribute name="NAME" x="86.36" y="27.94" size="1.016" layer="25" font="vector" ratio="10" align="center-left"/>
 </element>
-<element name="R9" library="rcl" package="R0603" value="10K" x="78.105" y="27.94" smashed="yes" rot="R180">
+<element name="R9" library="rcl" package="R0603" value="DNP" x="78.105" y="27.94" smashed="yes" rot="R180">
 <attribute name="NAME" x="80.01" y="27.94" size="1.016" layer="25" font="vector" ratio="10" align="center-left"/>
 </element>

Commit message: ES基板の回路図に部品の値を記入
Parts:
- VR1, VR2: value (none) -> 10K
Changed lines of the file:
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@@
 <attribute name="NAME" x="127.635" y="24.13" size="1.016" layer="25" font="vector" ratio="10" align="bottom-right"/>
 </element>
-<element name="VR1" library="pot-suntan" package="3386K" value="" x="58.42" y="17.78" smashed="yes">
+<element name="VR1" library="pot-suntan" package="3386K" value="10K" x="58.42" y="17.78" smashed="yes">
 <attribute name="NAME" x="53.975" y="22.86" size="1.016" layer="25" font="vector" ratio="10"/>
 <attribute name="VALUE" x="65.0875" y="14.2875" size="1.27" layer="27" ratio="12" rot="R90"/>
 </element>
-<element name="VR2" library="pot-suntan" package="3386T" value="" x="58.42" y="17.78" smashed="yes">
+<element name="VR2" library="pot-suntan" package="3386T" value="10K" x="58.42" y="17.78" smashed="yes">
 <attribute name="NAME" x="57.785" y="22.86" size="1.016" layer="25" font="vector" ratio="10"/>
 <attribute name="VALUE" x="65.0875" y="13.335" size="1.27" layer="27" ratio="12" rot="R90"/>

Commit message: ES基板の回路図に部品の値を記入
Parts:
- C9: value (none) -> 10u
- R12: value (none) -> 10K
- R13, R14: value (none) -> DNP
Changed lines of the file:
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@@
 <attribute name="NAME" x="80.01" y="33.02" size="1.016" layer="25" font="vector" ratio="10" align="center-left"/>
 </element>
-<element name="C9" library="rcl" package="C0805" value="" x="119.38" y="67.31" smashed="yes">
+<element name="C9" library="rcl" package="C0805" value="10u" x="119.38" y="67.31" smashed="yes">
 <attribute name="NAME" x="119.38" y="68.58" size="1.016" layer="25" font="vector" ratio="10" align="bottom-center"/>
 <attribute name="VALUE" x="118.11" y="64.77" size="1.27" layer="27"/>
@@
 <attribute name="NAME" x="80.01" y="30.48" size="1.016" layer="25" font="vector" ratio="10" align="center-left"/>
 </element>
-<element name="R12" library="rcl" package="R0603" value="" x="104.775" y="67.945" smashed="yes" rot="R180">
+<element name="R12" library="rcl" package="R0603" value="10K" x="104.775" y="67.945" smashed="yes" rot="R180">
 <attribute name="NAME" x="104.775" y="69.215" size="1.016" layer="25" font="vector" ratio="10" align="bottom-center"/>
 <attribute name="VALUE" x="105.41" y="69.85" size="1.27" layer="27" rot="R180"/>
 </element>
-<element name="R13" library="rcl" package="R0603" value="" x="112.395" y="25.4" smashed="yes">
+<element name="R13" library="rcl" package="R0603" value="DNP" x="112.395" y="25.4" smashed="yes">
 <attribute name="NAME" x="112.395" y="26.67" size="1.016" layer="25" font="vector" ratio="10" align="bottom-center"/>
 <attribute name="VALUE" x="111.76" y="23.495" size="1.27" layer="27"/>
 </element>
-<element name="R14" library="rcl" package="R0603" value="" x="116.205" y="25.4" smashed="yes" rot="R180">
+<element name="R14" library="rcl" package="R0603" value="DNP" x="116.205" y="25.4" smashed="yes" rot="R180">
 <attribute name="NAME" x="116.205" y="26.67" size="1.016" layer="25" font="vector" ratio="10" align="bottom-center"/>
 <attribute name="VALUE" x="116.84" y="27.305" size="1.27" layer="27" rot="R180"/>
