File: hardware/algyan_8th.es.sch (EAGLE design)
At the start: 40 parts, among them CN1 4P-2.0, U1 XIAO ESP32C3, U2 TM1640, U3 OSL641501-AY, U4 LTP-12188M-08, U5 NJM2113D, U6 UGSM23A, U7 EC12PLRVF, U8 TVGP01-G73BB, U9 TVGP01-G73BB

Commit message: ES基板の回路図に部品の値を記入
Parts:
- C1: value (none) -> 10u
- C3: value (none) -> DNP
- C7, C8: value 0.01u -> DNP
- R1, R2: value (none) -> 100K
- R10, R11: value 10K -> 0
- R5: value (none) -> 0
- R8, R9: value 10K -> DNP
Changed lines of the file:
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@@
 <part name="U5" library="matsujirushi" deviceset="NJM2113" device="D"/>
 <part name="U6" library="matsujirushi" deviceset="UGSM23A" device=""/>
-<part name="R1" library="rcl" deviceset="R-EU_" device="R0603"/>
-<part name="R2" library="rcl" deviceset="R-EU_" device="R0603"/>
+<part name="R1" library="rcl" deviceset="R-EU_" device="R0603" value="100K"/>
+<part name="R2" library="rcl" deviceset="R-EU_" device="R0603" value="100K"/>
 <part name="R3" library="rcl" deviceset="R-EU_" device="R0603" value="10K"/>
 <part name="R4" library="rcl" deviceset="R-EU_" device="R0603" value="10K"/>
@@
 <part name="VR2" library="pot-suntan" deviceset="3386-" device="T"/>
 <part name="U$5" library="Power or GND " deviceset="GND_POWER" device=""/>
-<part name="C3" library="rcl" deviceset="C-EU" device="C0805"/>
-<part name="R5" library="rcl" deviceset="R-EU_" device="R0603"/>
+<part name="C3" library="rcl" deviceset="C-EU" device="C0805" value="DNP"/>
+<part name="R5" library="rcl" deviceset="R-EU_" device="R0603" value="0"/>
 <part name="U$6" library="Power or GND " deviceset="GND_POWER" device=""/>
 <part name="U$7" library="Power or GND " deviceset="GND_POWER" device=""/>
-<part name="R8" library="rcl" deviceset="R-EU_" device="R0603" value="10K"/>
-<part name="R9" library="rcl" deviceset="R-EU_" device="R0603" value="10K"/>
-<part name="R10" library="rcl" deviceset="R-EU_" device="R0603" value="10K"/>
-<part name="R11" library="rcl" deviceset="R-EU_" device="R0603" value="10K"/>
-<part name="C7" library="rcl" deviceset="C-EU" device="C0603" value="0.01u"/>
-<part name="C8" library="rcl" deviceset="C-EU" device="C0603" value="0.01u"/>
+<part name="R8" library="rcl" deviceset="R-EU_" device="R0603" value="DNP"/>
+<part name="R9" library="rcl" deviceset="R-EU_" device="R0603" value="DNP"/>
+<part name="R10" library="rcl" deviceset="R-EU_" device="R0603" value="0"/>
+<part name="R11" library="rcl" deviceset="R-EU_" device="R0603" value="0"/>
+<part name="C7" library="rcl" deviceset="C-EU" device="C0603" value="DNP"/>
+<part name="C8" library="rcl" deviceset="C-EU" device="C0603" value="DNP"/>
 <part name="U$8" library="Power or GND " deviceset="GND_POWER" device=""/>
 <part name="U$9" library="Power or GND " deviceset="GND_POWER" device=""/>
@@
 <part name="U$15" library="Power or GND " deviceset="GND_POWER" device=""/>
 <part name="JP1" library="SparkFun-Jumpers" deviceset="JUMPER-SMT_3_NO" device="_SILK" value=""/>
-<part name="C1" library="rcl" deviceset="C-EU" device="C0805"/>
+<part name="C1" library="rcl" deviceset="C-EU" device="C0805" value="10u"/>
 <part name="CN1" library="Seeed-Connector" deviceset="GROVE-CONNECTOR-DIP(4P-2.0)" device="" value="4P-2.0"/>
 <part name="U$16" library="Power or GND " deviceset="GND_POWER" device=""/>

Commit message: ES基板の回路図に部品の値を記入
Parts:
- VR1, VR2: value (none) -> 10K
Changed lines of the file:
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@@
 <part name="R6" library="rcl" deviceset="R-EU_" device="R0603" value="DNP"/>
 <part name="U$4" library="Power or GND " deviceset="GND_POWER" device=""/>
-<part name="VR1" library="pot-suntan" deviceset="3386-" device="K"/>
-<part name="VR2" library="pot-suntan" deviceset="3386-" device="T"/>
+<part name="VR1" library="pot-suntan" deviceset="3386-" device="K" value="10K"/>
+<part name="VR2" library="pot-suntan" deviceset="3386-" device="T" value="10K"/>
 <part name="U$5" library="Power or GND " deviceset="GND_POWER" device=""/>
 <part name="C3" library="rcl" deviceset="C-EU" device="C0805" value="DNP"/>

Commit message: ES基板の回路図に部品の値を記入
Parts:
- C9: value (none) -> 10u
- R12: value (none) -> 10K
- R13, R14: value (none) -> DNP
Other:
- note added: "D6はリセット直後HIGH出力"
- note added: "D9はBOOTボタンに接続されている（アクティブLOW）"
Changed lines of the file:
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@@
 <setting verticaltext="up"/>
 </settings>
-<grid distance="0.1" unitdist="inch" unit="inch" style="lines" multiple="1" display="no" altdistance="0.01" altunitdist="inch" altunit="inch"/>
+<grid distance="0.1" unitdist="inch" unit="inch" style="lines" multiple="1" display="yes" altdistance="0.01" altunitdist="inch" altunit="inch"/>
 <layers>
 <layer number="1" name="Top" color="4" fill="1" visible="no" active="no"/>
@@
 <part name="U9" library="matsujirushi" deviceset="TVGP01-G73BB" device=""/>
 <part name="LED1" library="led" deviceset="LED" device="5MM"/>
-<part name="R12" library="rcl" deviceset="R-EU_" device="R0603"/>
+<part name="R12" library="rcl" deviceset="R-EU_" device="R0603" value="10K"/>
 <part name="U5" library="matsujirushi" deviceset="NJM2113" device="D"/>
 <part name="U6" library="matsujirushi" deviceset="UGSM23A" device=""/>
@@
 <part name="U$10" library="Power or GND " deviceset="GND_POWER" device=""/>
 <part name="U$11" library="Power or GND " deviceset="GND_POWER" device=""/>
-<part name="R13" library="rcl" deviceset="R-EU_" device="R0603"/>
-<part name="R14" library="rcl" deviceset="R-EU_" device="R0603"/>
+<part name="R13" library="rcl" deviceset="R-EU_" device="R0603" value="DNP"/>
+<part name="R14" library="rcl" deviceset="R-EU_" device="R0603" value="DNP"/>
 <part name="U$12" library="Power or GND " deviceset="GND_POWER" device=""/>
 <part name="U$13" library="Power or GND " deviceset="GND_POWER" device=""/>
@@
 <part name="CN1" library="Seeed-Connector" deviceset="GROVE-CONNECTOR-DIP(4P-2.0)" device="" value="4P-2.0"/>
 <part name="U$16" library="Power or GND " deviceset="GND_POWER" device=""/>
-<part name="C9" library="rcl" deviceset="C-EU" device="C0805"/>
+<part name="C9" library="rcl" deviceset="C-EU" device="C0805" value="10u"/>
 <part name="JP2" library="SparkFun-Jumpers" deviceset="JUMPER-SMT_2_NO" device="_SILK"/>
 <part name="JP3" library="SparkFun-Jumpers" deviceset="JUMPER-SMT_2_NO" device="_SILK"/>
@@
 <text x="198.12" y="43.18" size="1.778" layer="97" align="center-left">VCC</text>
 <text x="198.12" y="40.64" size="1.778" layer="97" align="center-left">GND</text>
+<text x="274.32" y="198.12" size="1.778" layer="97">D9はBOOTボタンに接続されている（アクティブLOW）</text>
+<text x="274.32" y="200.66" size="1.778" layer="97">D6はリセット直後HIGH出力</text>
 </plain>
 <instances>
