File: hardware/algyan_8th.es3.sch (EAGLE design)
At the start: 43 parts, among them CN1 4P-2.0, U1 XIAO ESP32C3, U10 EC12E(Panel), U2 TM1640, U3 NJM2113M, U4 LTP-12188M-08, U5 NJM2113D, U6 UGSM23A, U7 EC12PLRVF, U8 TVGP01-G73BB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

Commit message: ES3基板のEAGLEファイルと回路図PDFを追加
Parts:
- removed R17, R6: 0, rcl:R-EU_R0603
- added R18: 10K, rcl:R-EU_R0603
- JP2: value JUMPER-SMT_3_1-NC_TRACE_SILK -> JUMPER-SMT_3_NO_SILK; device SparkFun-Jumpers:JUMPER-SMT_3_1-NC_TRACE_SILK -> SparkFun-Jumpers:JUMPER-SMT_3_NO_SILK
- R1, R2: value 100K -> 10K
- R7: value (none) -> 10K
Connections:
- removed net N$17: CN1.1, R15.1, R6.1
- removed net N$18: CN1.2, R16.1, R17.1
- net LED: now also R18.1
- net N$6: now also R18.2
- net SCL: now also CN1.1, R15.1; no longer R6.2
- net SDA: now also CN1.2, R16.1; no longer R17.2
Other:
- note added: "JP2をNOに変更"
- note added: "R1とR2を10K"
- note added: "SCL/SDAのダンピング抵抗を削除"
- note added: "ロータリーエンコーダLEDの電流制限抵抗を2個並列に"
- moved on the sheet: R7
Changed lines of the file:
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@@
 <part name="U5" library="matsujirushi" deviceset="NJM2113" device="D"/>
 <part name="U6" library="matsujirushi" deviceset="UGSM23A" device=""/>
-<part name="R1" library="rcl" deviceset="R-EU_" device="R0603" value="100K"/>
-<part name="R2" library="rcl" deviceset="R-EU_" device="R0603" value="100K"/>
+<part name="R1" library="rcl" deviceset="R-EU_" device="R0603" value="10K"/>
+<part name="R2" library="rcl" deviceset="R-EU_" device="R0603" value="10K"/>
 <part name="R3" library="rcl" deviceset="R-EU_" device="R0603" value="10K"/>
 <part name="R4" library="rcl" deviceset="R-EU_" device="R0603" value="10K"/>
@@
 <part name="U$8" library="Power or GND " deviceset="GND_POWER" device=""/>
 <part name="U$9" library="Power or GND " deviceset="GND_POWER" device=""/>
-<part name="R7" library="rcl" deviceset="R-EU_" device="R0603"/>
+<part name="R7" library="rcl" deviceset="R-EU_" device="R0603" value="10K"/>
 <part name="R13" library="rcl" deviceset="R-EU_" device="R0603" value="DNP"/>
 <part name="R14" library="rcl" deviceset="R-EU_" device="R0603" value="DNP"/>
@@
 <part name="R16" library="rcl" deviceset="R-EU_" device="R0603" value="DNP"/>
 <part name="U3" library="matsujirushi" deviceset="NJM2113" device="M" value="NJM2113M"/>
-<part name="JP2" library="SparkFun-Jumpers" deviceset="JUMPER-SMT_3_1-NC_TRACE" device="_SILK"/>
 <part name="JP3" library="pinhead" deviceset="PINHD-1X1" device=""/>
-<part name="R6" library="rcl" deviceset="R-EU_" device="R0603" value="0"/>
-<part name="R17" library="rcl" deviceset="R-EU_" device="R0603" value="0"/>
+<part name="JP2" library="SparkFun-Jumpers" deviceset="JUMPER-SMT_3_NO" device="_SILK"/>
+<part name="R18" library="rcl" deviceset="R-EU_" device="R0603" value="10K"/>
 </parts>
 <sheets>
@@
 <text x="340.36" y="256.54" size="1.778" layer="97">SPEAKER-ENABLEとLEDのピン割当を入れ替え</text>
 <text x="340.36" y="254" size="1.778" layer="97">SELECT-BTNとESCAPE-BTNの信号名を変更</text>
+<text x="340.36" y="251.46" size="1.778" layer="97">SCL/SDAのダンピング抵抗を削除</text>
+<text x="340.36" y="248.92" size="1.778" layer="97">ロータリーエンコーダLEDの電流制限抵抗を2個並列に</text>
+<text x="340.36" y="246.38" size="1.778" layer="97">JP2をNOに変更</text>
+<text x="340.36" y="243.84" size="1.778" layer="97">R1とR2を10K</text>
 </plain>
 <instances>
@@
 <instance part="U$8" gate="G$1" x="129.54" y="40.64" smashed="yes"/>
 <instance part="U$9" gate="G$1" x="139.7" y="40.64" smashed="yes"/>
-<instance part="R7" gate="G$1" x="55.88" y="27.94" rot="R90"/>
+<instance part="R7" gate="G$1" x="48.26" y="27.94" rot="R90"/>
 <instance part="R13" gate="G$1" x="302.26" y="160.02" rot="R90"/>
 <instance part="R14" gate="G$1" x="320.04" y="160.02" rot="R90"/>
@@
 <instance part="U3" gate="-1" x="78.74" y="104.14" rot="MR0"/>
 <instance part="U3" gate="-2" x="325.12" y="73.66"/>
+<instance part="JP3" gate="G$1" x="276.86" y="185.42"/>
 <instance part="JP2" gate="G$1" x="261.62" y="185.42" smashed="yes" rot="R270">
 <attribute name="NAME" x="262.001" y="182.88" size="1.778" layer="95" font="vector" rot="R270"/>
 </instance>
-<instance part="JP3" gate="G$1" x="276.86" y="185.42"/>
-<instance part="R6" gate="G$1" x="241.3" y="48.26"/>
-<instance part="R17" gate="G$1" x="241.3" y="45.72"/>
+<instance part="R18" gate="G$1" x="55.88" y="27.94" rot="R90"/>
 </instances>
 <busses>
@@
 <bus name="SCL,SDA">
 <segment>
-<wire x1="256.54" y1="45.72" x2="256.54" y2="73.66" width="0.762" layer="92"/>
-<wire x1="256.54" y1="73.66" x2="246.38" y2="73.66" width="0.762" layer="92"/>
-<wire x1="246.38" y1="73.66" x2="246.38" y2="213.36" width="0.762" layer="92"/>
+<wire x1="246.38" y1="45.72" x2="246.38" y2="213.36" width="0.762" layer="92"/>
 </segment>
 </bus>
@@
 </segment>
 <segment>
-<pinref part="JP2" gate="G$1" pin="3"/>
 <wire x1="220.98" y1="185.42" x2="256.54" y2="185.42" width="0.1524" layer="91"/>
 <label x="223.52" y="185.42" size="1.778" layer="95"/>
+<pinref part="JP2" gate="G$1" pin="3"/>
 </segment>
 </net>
@@
 <segment>
 <wire x1="177.8" y1="20.32" x2="55.88" y2="20.32" width="0.1524" layer="91"/>
-<wire x1="55.88" y1="20.32" x2="55.88" y2="22.86" width="0.1524" layer="91"/>
+<wire x1="55.88" y1="20.32" x2="48.26" y2="20.32" width="0.1524" layer="91"/>
+<wire x1="48.26" y1="20.32" x2="48.26" y2="22.86" width="0.1524" layer="91"/>
 <label x="175.26" y="20.32" size="1.778" layer="95" rot="MR0"/>
 <pinref part="R7" gate="G$1" pin="1"/>
+<pinref part="R18" gate="G$1" pin="1"/>
+<wire x1="55.88" y1="22.86" x2="55.88" y2="20.32" width="0.1524" layer="91"/>
+<junction x="55.88" y="20.32"/>
 </segment>
 <segment>
@@
 </segment>
 <segment>
-<pinref part="R17" gate="G$1" pin="2"/>
-<wire x1="256.54" y1="45.72" x2="246.38" y2="45.72" width="0.1524" layer="91"/>
-<label x="254" y="45.72" size="1.778" layer="95" rot="MR0"/>
+<label x="243.84" y="45.72" size="1.778" layer="95" rot="MR0"/>
+<pinref part="CN1" gate="G$1" pin="2"/>
+<wire x1="208.28" y1="45.72" x2="223.52" y2="45.72" width="0.1524" layer="91"/>
+<pinref part="R16" gate="G$1" pin="1"/>
+<wire x1="223.52" y1="45.72" x2="246.38" y2="45.72" width="0.1524" layer="91"/>
+<wire x1="223.52" y1="50.8" x2="223.52" y2="45.72" width="0.1524" layer="91"/>
+<junction x="223.52" y="45.72"/>
 </segment>
 </net>
@@
 </segment>
 <segment>
-<pinref part="R6" gate="G$1" pin="2"/>
-<wire x1="256.54" y1="48.26" x2="246.38" y2="48.26" width="0.1524" layer="91"/>
-<label x="254" y="48.26" size="1.778" layer="95" rot="MR0"/>
+<label x="243.84" y="48.26" size="1.778" layer="95" rot="MR0"/>
+<pinref part="CN1" gate="G$1" pin="1"/>
+<wire x1="208.28" y1="48.26" x2="215.9" y2="48.26" width="0.1524" layer="91"/>
+<pinref part="R15" gate="G$1" pin="1"/>
+<wire x1="215.9" y1="48.26" x2="246.38" y2="48.26" width="0.1524" layer="91"/>
+<wire x1="215.9" y1="50.8" x2="215.9" y2="48.26" width="0.1524" layer="91"/>
+<junction x="215.9" y="48.26"/>
 </segment>
 </net>
@@
 <segment>
 <pinref part="R7" gate="G$1" pin="2"/>
+<wire x1="48.26" y1="33.02" x2="48.26" y2="35.56" width="0.1524" layer="91"/>
+<pinref part="U7" gate="G$1" pin="LED-"/>
+<wire x1="48.26" y1="35.56" x2="55.88" y2="35.56" width="0.1524" layer="91"/>
+<pinref part="R18" gate="G$1" pin="2"/>
+<wire x1="55.88" y1="35.56" x2="60.96" y2="35.56" width="0.1524" layer="91"/>
 <wire x1="55.88" y1="33.02" x2="55.88" y2="35.56" width="0.1524" layer="91"/>
-<pinref part="U7" gate="G$1" pin="LED-"/>
-<wire x1="55.88" y1="35.56" x2="60.96" y2="35.56" width="0.1524" layer="91"/>
+<junction x="55.88" y="35.56"/>
 </segment>
 </net>
@@
 <net name="N$16" class="0">
 <segment>
-<pinref part="JP2" gate="G$1" pin="1"/>
 <wire x1="266.7" y1="185.42" x2="274.32" y2="185.42" width="0.1524" layer="91"/>
 <pinref part="JP3" gate="G$1" pin="1"/>
-</segment>
-</net>
-<net name="N$17" class="0">
-<segment>
-<pinref part="CN1" gate="G$1" pin="1"/>
-<pinref part="R6" gate="G$1" pin="1"/>
-<wire x1="208.28" y1="48.26" x2="215.9" y2="48.26" width="0.1524" layer="91"/>
-<pinref part="R15" gate="G$1" pin="1"/>
-<wire x1="215.9" y1="48.26" x2="236.22" y2="48.26" width="0.1524" layer="91"/>
-<wire x1="215.9" y1="50.8" x2="215.9" y2="48.26" width="0.1524" layer="91"/>
-<junction x="215.9" y="48.26"/>
-</segment>
-</net>
-<net name="N$18" class="0">
-<segment>
-<pinref part="CN1" gate="G$1" pin="2"/>
-<pinref part="R17" gate="G$1" pin="1"/>
-<wire x1="208.28" y1="45.72" x2="223.52" y2="45.72" width="0.1524" layer="91"/>
-<pinref part="R16" gate="G$1" pin="1"/>
-<wire x1="223.52" y1="45.72" x2="236.22" y2="45.72" width="0.1524" layer="91"/>
-<wire x1="223.52" y1="50.8" x2="223.52" y2="45.72" width="0.1524" layer="91"/>
-<junction x="223.52" y="45.72"/>
-</segment>
-</net>
+<pinref part="JP2" gate="G$1" pin="1"/>
+</segment>
+</net>
