File: hardware/xiaogyan.v1.brd (EAGLE design)
At the start: 142 x 55 mm, 42 parts, among them CN1 4P-2.0, U1 XIAO ESP32C3, U10 TVGP01-G73BB, U11 10K, U12 10K, U13 DNP, U2 TM1640, U3 LTP-12188M-08, U4 NJM2113D, U5 NJM2113M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

Commit message: R7とC6を変更
Parts:
- C6: value DNP -> 1000p
- R7: value 0 -> 10K
Changed lines of the file:
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@@
 <attribute name="NAME" x="86.36" y="8.89" size="1.016" layer="25" font="vector" ratio="10" rot="R90" align="bottom-center"/>
 </element>
-<element name="C6" library="rcl" package="C0805" value="DNP" x="72.39" y="5.715" smashed="yes" rot="R270">
+<element name="C6" library="rcl" package="C0805" value="1000p" x="72.39" y="5.715" smashed="yes" rot="R270">
 <attribute name="NAME" x="71.12" y="5.715" size="1.016" layer="25" font="vector" ratio="10" rot="R90" align="bottom-center"/>
 </element>
@@
 <attribute name="NAME" x="86.36" y="5.08" size="1.016" layer="25" font="vector" ratio="10" rot="R90" align="bottom-center"/>
 </element>
-<element name="R7" library="rcl" package="R0603" value="0" x="72.39" y="10.16" smashed="yes" rot="R90">
+<element name="R7" library="rcl" package="R0603" value="10K" x="72.39" y="10.16" smashed="yes" rot="R90">
 <attribute name="NAME" x="71.12" y="10.16" size="1.016" layer="25" font="vector" ratio="10" rot="R90" align="bottom-center"/>
 </element>
