File: hardware/xiaogyan.v1.sch (EAGLE design)
At the start: 42 parts, among them CN1 4P-2.0, U1 XIAO ESP32C3, U10 TVGP01-G73BB, U11 10K, U12 10K, U13 DNP, U2 TM1640, U3 LTP-12188M-08, U4 NJM2113D, U5 NJM2113M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

Commit message: R7とC6を変更
Parts:
- C6: value DNP -> 1000p
- R7: value 0 -> 10K
Changed lines of the file:
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@@
 <part name="U12" library="pot-suntan" deviceset="3386-" device="T" value="10K"/>
 <part name="U$5" library="Power or GND " deviceset="GND_POWER" device=""/>
-<part name="C6" library="rcl" deviceset="C-EU" device="C0805" value="DNP"/>
-<part name="R7" library="rcl" deviceset="R-EU_" device="R0603" value="0"/>
+<part name="C6" library="rcl" deviceset="C-EU" device="C0805" value="1000p"/>
+<part name="R7" library="rcl" deviceset="R-EU_" device="R0603" value="10K"/>
 <part name="U$6" library="Power or GND " deviceset="GND_POWER" device=""/>
 <part name="U$7" library="Power or GND " deviceset="GND_POWER" device=""/>
